File: XBee_SX_Pro_breakout/xbee_sx_pro_breakout/xbee_pro_sx_breakout_1.brd (EAGLE design)
At the start: 48 x 36 mm, 4 parts

Commit message: finished breakout board
Connections:
- removed net N$38: J2.14, U$1.38
- new net GND: J2.14, U$1.38
Routing:
- net N$38: track 14.9 -> 0.00 mm
- net GND: track 0.00 -> 14.9 mm, vias 6 -> 49
Changed lines of the file:
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@@
 <contactref element="U$1" pad="1"/>
 <contactref element="J2" pad="13"/>
-<wire x1="34.7472" y1="29.2608" x2="34.1376" y2="29.2608" width="0.1524" layer="1"/>
-<wire x1="38.862" y1="33.3756" x2="34.7472" y2="29.2608" width="0.1524" layer="1"/>
+<wire x1="34.2472" y1="29.2608" x2="34.1376" y2="29.2608" width="0.1524" layer="1"/>
+<wire x1="38.082184375" y1="33.095784375" x2="34.2472" y2="29.2608" width="0.1524" layer="1"/>
 <wire x1="34.1376" y1="29.2608" x2="34" y2="29.25" width="0.1524" layer="1"/>
-<wire x1="38.862" y1="33.3756" x2="38.93" y2="33.4" width="0.1524" layer="1"/>
-</signal>
-<signal name="N$38">
-<contactref element="U$1" pad="38"/>
-<contactref element="J2" pad="14"/>
-<wire x1="41.4528" y1="33.528" x2="31.0896" y2="23.1648" width="0.1524" layer="1"/>
-<wire x1="31.0896" y1="23.1648" x2="31" y2="23.15" width="0.1524" layer="1"/>
-<wire x1="41.4528" y1="33.528" x2="41.47" y2="33.4" width="0.1524" layer="1"/>
+<wire x1="38.082184375" y1="33.095784375" x2="38.93" y2="33.4" width="0.1524" layer="1"/>
 </signal>
 <signal name="GND">
@@
 <via x="18" y="25" extent="1-16" drill="0.35"/>
 <via x="21" y="25" extent="1-16" drill="0.35"/>
-</signal>
-<signal name="N$43">
 <via x="24" y="25" extent="1-16" drill="0.35"/>
-</signal>
-<signal name="N$44">
 <via x="27" y="25" extent="1-16" drill="0.35"/>
-</signal>
-<signal name="N$45">
+<via x="31" y="26" extent="1-16" drill="0.35"/>
 <via x="35" y="25" extent="1-16" drill="0.35"/>
-</signal>
-<signal name="N$46">
 <via x="38" y="25" extent="1-16" drill="0.35"/>
-</signal>
-<signal name="N$47">
+<via x="38" y="22" extent="1-16" drill="0.35"/>
+<via x="35" y="22" extent="1-16" drill="0.35"/>
+<via x="27" y="22" extent="1-16" drill="0.35"/>
+<via x="24" y="22" extent="1-16" drill="0.35"/>
+<via x="21" y="22" extent="1-16" drill="0.35"/>
+<via x="18" y="22" extent="1-16" drill="0.35"/>
+<via x="15" y="22" extent="1-16" drill="0.35"/>
 <via x="12" y="22" extent="1-16" drill="0.35"/>
-</signal>
-<signal name="N$48">
-<via x="15" y="22" extent="1-16" drill="0.35"/>
-</signal>
-<signal name="N$49">
-<via x="18" y="22" extent="1-16" drill="0.35"/>
-</signal>
-<signal name="N$50">
-<via x="21" y="22" extent="1-16" drill="0.35"/>
-</signal>
-<signal name="N$51">
-<via x="24" y="22" extent="1-16" drill="0.35"/>
-</signal>
-<signal name="N$52">
-<via x="27" y="22" extent="1-16" drill="0.35"/>
-</signal>
-<signal name="N$53">
 <via x="12" y="19" extent="1-16" drill="0.35"/>
-</signal>
-<signal name="N$54">
 <via x="15" y="19" extent="1-16" drill="0.35"/>
-</signal>
-<signal name="N$55">
 <via x="18" y="19" extent="1-16" drill="0.35"/>
-</signal>
-<signal name="N$56">
 <via x="21" y="19" extent="1-16" drill="0.35"/>
-</signal>
-<signal name="N$57">
 <via x="24" y="19" extent="1-16" drill="0.35"/>
-</signal>
-<signal name="N$58">
 <via x="27" y="19" extent="1-16" drill="0.35"/>
-</signal>
-<signal name="N$59">
+<via x="31" y="19" extent="1-16" drill="0.35"/>
+<via x="35" y="19" extent="1-16" drill="0.35"/>
+<via x="38" y="19" extent="1-16" drill="0.35"/>
 <via x="12" y="16" extent="1-16" drill="0.35"/>
-</signal>
-<signal name="N$60">
 <via x="15" y="16" extent="1-16" drill="0.35"/>
-</signal>
-<signal name="N$61">
 <via x="18" y="16" extent="1-16" drill="0.35"/>
-</signal>
-<signal name="N$62">
 <via x="21" y="16" extent="1-16" drill="0.35"/>
-</signal>
-<signal name="N$63">
 <via x="24" y="16" extent="1-16" drill="0.35"/>
-</signal>
-<signal name="N$64">
 <via x="27" y="16" extent="1-16" drill="0.35"/>
-</signal>
-<signal name="N$65">
+<via x="31" y="16" extent="1-16" drill="0.35"/>
+<via x="35" y="16" extent="1-16" drill="0.35"/>
+<via x="38" y="16" extent="1-16" drill="0.35"/>
+<via x="38" y="13" extent="1-16" drill="0.35"/>
+<via x="38" y="10" extent="1-16" drill="0.35"/>
+<via x="27" y="13" extent="1-16" drill="0.35"/>
+<via x="24" y="13" extent="1-16" drill="0.35"/>
+<via x="21" y="13" extent="1-16" drill="0.35"/>
+<via x="24" y="10" extent="1-16" drill="0.35"/>
+<via x="21" y="10" extent="1-16" drill="0.35"/>
+<via x="18" y="10" extent="1-16" drill="0.35"/>
+<via x="18" y="13" extent="1-16" drill="0.35"/>
+<via x="15" y="13" extent="1-16" drill="0.35"/>
 <via x="12" y="13" extent="1-16" drill="0.35"/>
-</signal>
-<signal name="N$66">
-<via x="15" y="13" extent="1-16" drill="0.35"/>
-</signal>
-<signal name="N$67">
-<via x="18" y="13" extent="1-16" drill="0.35"/>
-</signal>
-<signal name="N$68">
-<via x="21" y="13" extent="1-16" drill="0.35"/>
-</signal>
-<signal name="N$69">
-<via x="24" y="13" extent="1-16" drill="0.35"/>
-</signal>
-<signal name="N$70">
-<via x="27" y="13" extent="1-16" drill="0.35"/>
-</signal>
-<signal name="N$71">
 <via x="12" y="10" extent="1-16" drill="0.35"/>
-</signal>
-<signal name="N$73">
-<via x="18" y="10" extent="1-16" drill="0.35"/>
-</signal>
-<signal name="N$74">
-<via x="21" y="10" extent="1-16" drill="0.35"/>
-</signal>
-<signal name="N$75">
-<via x="24" y="10" extent="1-16" drill="0.35"/>
-</signal>
-<signal name="N$77">
-<via x="35" y="22" extent="1-16" drill="0.35"/>
-</signal>
-<signal name="N$78">
-<via x="38" y="22" extent="1-16" drill="0.35"/>
-</signal>
-<signal name="N$79">
-<via x="35" y="19" extent="1-16" drill="0.35"/>
-</signal>
-<signal name="N$80">
-<via x="38" y="19" extent="1-16" drill="0.35"/>
-</signal>
-<signal name="N$81">
-<via x="35" y="16" extent="1-16" drill="0.35"/>
-</signal>
-<signal name="N$82">
-<via x="38" y="16" extent="1-16" drill="0.35"/>
-</signal>
-<signal name="N$83">
-<via x="38" y="13" extent="1-16" drill="0.35"/>
-</signal>
-<signal name="N$84">
-<via x="38" y="10" extent="1-16" drill="0.35"/>
-</signal>
-<signal name="N$85">
-<via x="31" y="19" extent="1-16" drill="0.35"/>
-</signal>
-<signal name="N$86">
-<via x="31" y="16" extent="1-16" drill="0.35"/>
-</signal>
-<signal name="N$87">
-<via x="31" y="25" extent="1-16" drill="0.35"/>
+<contactref element="U$1" pad="38"/>
+<contactref element="J2" pad="14"/>
+<wire x1="41.4528" y1="33.528" x2="31.0896" y2="23.1648" width="0.1524" layer="1"/>
+<wire x1="31.0896" y1="23.1648" x2="31" y2="23.15" width="0.1524" layer="1"/>
+<wire x1="41.4528" y1="33.528" x2="41.47" y2="33.4" width="0.1524" layer="1"/>
 </signal>
 </signals>

Commit message: updated gnd signals
Connections:
- net N$36 renamed VCC
- removed net N$16: J3.16, U$1.22
- removed net N$25: J2.1, U$1.13
- removed net N$27: J2.3, U$1.11
- removed net N$3: J3.3, U$1.35
- removed net N$37: J2.13, U$1.1
- net GND: now also J2.1, J2.13, J2.3, J3.16, J3.3, U$1.1, U$1.11, U$1.13, U$1.22, U$1.35
Routing:
- net N$37: track 6.57 -> 0.00 mm
- net N$3: track 6.36 -> 0.00 mm
- net N$16: track 5.63 -> 0.00 mm
- net N$25: track 4.87 -> 0.00 mm
- net N$27: track 4.41 -> 0.00 mm
- net GND: track 14.9 -> 17.1 mm
Changed lines of the file:
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@@
 <wire x1="42.672" y1="2.8956" x2="42.71" y2="2.8" width="0.1524" layer="1"/>
-</signal>
-<signal name="N$3">
-<contactref element="U$1" pad="35"/>
-<contactref element="J3" pad="3"/>
-<wire x1="36.1188" y1="6.5532" x2="36.1188" y2="7.1628" width="0.1524" layer="1"/>
-<wire x1="39.7764" y1="2.8956" x2="36.1188" y2="6.5532" width="0.1524" layer="1"/>
-<wire x1="40.0812" y1="2.8956" x2="39.7764" y2="2.8956" width="0.1524" layer="1"/>
-<wire x1="36.1188" y1="7.1628" x2="36" y2="7.25" width="0.1524" layer="1"/>
-<wire x1="40.0812" y1="2.8956" x2="40.17" y2="2.8" width="0.1524" layer="1"/>
 </signal>
 <signal name="N$4">
@@
 <wire x1="9.7536" y1="2.8956" x2="9.69" y2="2.8" width="0.1524" layer="1"/>
 </signal>
-<signal name="N$16">
-<contactref element="U$1" pad="22"/>
-<contactref element="J3" pad="16"/>
-<wire x1="9.906" y1="5.6388" x2="9.906" y2="7.1628" width="0.1524" layer="1"/>
-<wire x1="7.1628" y1="2.8956" x2="9.906" y2="5.6388" width="0.1524" layer="1"/>
-<wire x1="9.906" y1="7.1628" x2="10" y2="7.25" width="0.1524" layer="1"/>
-<wire x1="7.1628" y1="2.8956" x2="7.15" y2="2.8" width="0.1524" layer="1"/>
-</signal>
 <signal name="N$17">
 <contactref element="U$1" pad="21"/>
@@
 <wire x1="3.048" y1="27.1272" x2="3" y2="27.23" width="0.1524" layer="1"/>
 </signal>
-<signal name="N$25">
-<contactref element="U$1" pad="13"/>
-<contactref element="J2" pad="1"/>
-<wire x1="9.906" y1="32.004" x2="9.906" y2="29.2608" width="0.1524" layer="1"/>
-<wire x1="8.5344" y1="33.3756" x2="9.906" y2="32.004" width="0.1524" layer="1"/>
-<wire x1="9.906" y1="29.2608" x2="10" y2="29.25" width="0.1524" layer="1"/>
-<wire x1="8.5344" y1="33.3756" x2="8.45" y2="33.4" width="0.1524" layer="1"/>
-</signal>
 <signal name="N$26">
 <contactref element="U$1" pad="12"/>
@@
 <wire x1="11.8872" y1="29.2608" x2="12" y2="29.25" width="0.1524" layer="1"/>
 <wire x1="11.1252" y1="33.3756" x2="10.99" y2="33.4" width="0.1524" layer="1"/>
-</signal>
-<signal name="N$27">
-<contactref element="U$1" pad="11"/>
-<contactref element="J2" pad="3"/>
-<wire x1="13.8684" y1="33.0708" x2="13.8684" y2="29.2608" width="0.1524" layer="1"/>
-<wire x1="13.5636" y1="33.3756" x2="13.8684" y2="33.0708" width="0.1524" layer="1"/>
-<wire x1="13.8684" y1="29.2608" x2="14" y2="29.25" width="0.1524" layer="1"/>
-<wire x1="13.5636" y1="33.3756" x2="13.53" y2="33.4" width="0.1524" layer="1"/>
 </signal>
 <signal name="N$28">
@@
 <wire x1="33.8328" y1="33.3756" x2="33.85" y2="33.4" width="0.1524" layer="1"/>
 </signal>
-<signal name="N$36">
+<signal name="VCC">
 <contactref element="U$1" pad="2"/>
 <contactref element="J2" pad="12"/>
@@
 <wire x1="33.0085375" y1="31.2088" x2="33.9588" y2="31.2088" width="0.8128" layer="1"/>
 <wire x1="33.9588" y1="31.2088" x2="36.1256" y2="33.3756" width="0.8128" layer="1"/>
-</signal>
-<signal name="N$37">
-<contactref element="U$1" pad="1"/>
-<contactref element="J2" pad="13"/>
-<wire x1="34.2472" y1="29.2608" x2="34.1376" y2="29.2608" width="0.1524" layer="1"/>
-<wire x1="38.082184375" y1="33.095784375" x2="34.2472" y2="29.2608" width="0.1524" layer="1"/>
-<wire x1="34.1376" y1="29.2608" x2="34" y2="29.25" width="0.1524" layer="1"/>
-<wire x1="38.082184375" y1="33.095784375" x2="38.93" y2="33.4" width="0.1524" layer="1"/>
 </signal>
 <signal name="GND">
@@
 <contactref element="U$1" pad="38"/>
 <contactref element="J2" pad="14"/>
-<wire x1="41.4528" y1="33.528" x2="31.0896" y2="23.1648" width="0.1524" layer="1"/>
 <wire x1="31.0896" y1="23.1648" x2="31" y2="23.15" width="0.1524" layer="1"/>
 <wire x1="41.4528" y1="33.528" x2="41.47" y2="33.4" width="0.1524" layer="1"/>
+<contactref element="U$1" pad="13"/>
+<contactref element="J2" pad="1"/>
+<wire x1="9.906" y1="29.2608" x2="10" y2="29.25" width="0.1524" layer="1"/>
+<wire x1="8.5344" y1="33.3756" x2="8.45" y2="33.4" width="0.1524" layer="1"/>
+<contactref element="U$1" pad="1"/>
+<contactref element="J2" pad="13"/>
+<wire x1="34.2472" y1="29.2608" x2="34.1376" y2="29.2608" width="0.1524" layer="1"/>
+<wire x1="34.1376" y1="29.2608" x2="34" y2="29.25" width="0.1524" layer="1"/>
+<contactref element="U$1" pad="22"/>
+<contactref element="J3" pad="16"/>
+<wire x1="9.906" y1="5.6388" x2="9.906" y2="7.1628" width="0.1524" layer="1"/>
+<wire x1="7.1628" y1="2.8956" x2="9.906" y2="5.6388" width="0.1524" layer="1"/>
+<wire x1="9.906" y1="7.1628" x2="10" y2="7.25" width="0.1524" layer="1"/>
+<wire x1="7.1628" y1="2.8956" x2="7.15" y2="2.8" width="0.1524" layer="1"/>
+<contactref element="U$1" pad="35"/>
+<contactref element="J3" pad="3"/>
+<wire x1="36.1188" y1="6.5532" x2="36.1188" y2="7.1628" width="0.1524" layer="1"/>
+<wire x1="39.7764" y1="2.8956" x2="36.1188" y2="6.5532" width="0.1524" layer="1"/>
+<wire x1="40.0812" y1="2.8956" x2="39.7764" y2="2.8956" width="0.1524" layer="1"/>
+<wire x1="36.1188" y1="7.1628" x2="36" y2="7.25" width="0.1524" layer="1"/>
+<wire x1="40.0812" y1="2.8956" x2="40.17" y2="2.8" width="0.1524" layer="1"/>
+<contactref element="U$1" pad="11"/>
+<contactref element="J2" pad="3"/>
+<wire x1="13.8684" y1="33.0708" x2="13.8684" y2="29.2608" width="0.1524" layer="1"/>
+<wire x1="13.5636" y1="33.3756" x2="13.8684" y2="33.0708" width="0.1524" layer="1"/>
+<wire x1="13.8684" y1="29.2608" x2="14" y2="29.25" width="0.1524" layer="1"/>
+<wire x1="13.5636" y1="33.3756" x2="13.53" y2="33.4" width="0.1524" layer="1"/>
 </signal>
 </signals>
