File: libraries/schematic_v1.brd (EAGLE design)
At the start: 65 x 70 mm, 46 parts, among them Q1 BSS138, Q2 BSS138, Q3 BSS138, Q4 BSS138

Commit message: pushing
Parts:
- removed U$1: DEV-16771, teensy_4_1:DEV-16771
- added B1: ARDUINO_UNO_R3, SparkFun-Boards:ARDUINO_R3
- added R18: 10k, SparkFun-Resistors:0603
- added R19: 8.2k, SparkFun-Resistors:0603
- added U$4: TEENSY41-E, teensy:TENNSY41-E
Connections:
- removed net 3.3V: U$1.3.3V@1, U$1.3.3V@2
- removed net 5V: U$1.5V
- removed net G: U$1.G
- removed net N$9: JP1.10, U$1.D33
- removed net USB_GND1: U$1.USB_GND
- removed net USB_GND2: U$1.USB_GND@2
- removed net VBAT: U$1.VBAT
- removed net VUSB: U$1.VUSB
- new net N$15: U$4.37-PWM
- new net POWER_DIVIDED: R18.1, R19.2, U$4.27-A13/SCK1
- net +15V: now also R18.2
- net +5V: now also B1.VIN, U$4.VIN; no longer U$1.VIN
- net GND: now also B1.GND@1, R19.1, U$4.+5V, U$4.GND1, U$4.GND2, U$4.GND3, U$4.GND4, U$4.GND5, U$4.GND6; no longer U$1.AGND, U$1.GND, U$1.GND@1, U$1.GND@2
- net N$1: now also U$4.35-TX8; no longer U$1.D35
- net N$11: now also U$4.1-TX1/MISO1/CTX2; no longer U$1.D1
- net N$2: now also U$4.34-RX8; no longer U$1.D34
- net N$5: now also U$4.0-RX1/CS1/CRX2; no longer U$1.D0
- net RESET_: now also JP1.10, U$4.33-MCLK2; no longer U$1.D36
- net SCL: now also U$4.16-A2/RX4/SCL1; no longer U$1.D20/A6
- net SDA: now also U$4.17-A3/TX4/SDA1; no longer U$1.D19/A5
- net TEENSY_3.3V: no longer U$1.3.3V
Routing:
- net +5V: track 0.00 -> 189.4 mm
- net +15V: track 0.00 -> 99.8 mm, vias 0 -> 3
- net POWER_DIVIDED: track 0.00 -> 86.1 mm, vias 0 -> 1
- net RESET_: track 0.00 -> 68.3 mm
- net N$5: track 0.00 -> 59.6 mm, vias 0 -> 2
- net N$2: track 0.00 -> 59.2 mm
- net +3.3V: track 0.00 -> 57.0 mm, vias 0 -> 1
- net N$1: track 0.00 -> 55.3 mm
- net GND: track 0.00 -> 52.0 mm
- net N$11: track 0.00 -> 48.7 mm, vias 0 -> 1
- net TEENSY_3.3V: track 0.00 -> 30.5 mm
- net SCL: track 0.00 -> 25.1 mm, vias 0 -> 1
- net N$3: track 0.00 -> 24.4 mm
- net CAN_RX1: track 0.00 -> 22.7 mm, vias 0 -> 2
- net CAN_TX1: track 0.00 -> 22.6 mm, vias 0 -> 1
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- removed copper zone on layer 16, net GND
Other:
- board size 65 x 70 mm -> 120 x 70 mm
