File: processing_board/processing_board/schematic_v1.brd (EAGLE design)
At the start: 126 x 72 mm, 64 parts, among them IC1 74HC165D, Q1 BSS138, Q2 BSS138, Q3 BSS138, Q4 BSS138

Commit message: 3/5 updates
Parts:
- added J1: (no value), SparkFun-Connectors:1X02
- added J6: (no value), SparkFun-Connectors:1X08
- added J7, J8: (no value), SparkFun-Connectors:1X06_NO_SILK
- added U$5: ARDUINOUNO, adafruit:ARDUINO
- added U1: TJA1050, TJA1050:SOT96-1
- J3: device SparkFun-Connectors:1X04 -> SparkFun-Connectors:1X08
- moved J3 116.6 mm to (119.8, 28.4)
- moved U$1 81.0 mm to (37.0, 28.0)
- moved R17 79.5 mm to (33.0, 25.4), turned to 180 degrees
- moved D8 78.6 mm to (28.5, 25.5)
- moved IC1 3.00 mm to (29.0, 41.0)
- moved J5 3.00 mm to (-1.00, 62.0)
- moved S1 1.41 mm to (18.0, 60.0)
Connections:
- new net 3V: U$5.3V
- new net 5V: U$5.5V
- new net GND1: U$5.GND1
- new net GND2: U$5.GND2
- new net N$1: J1.2, U1.6
- new net N$2: J1.1, U1.7
- new net VIN: U$5.VIN
- net +3.3V: now also J8.5
- net +5V: now also J8.1, J8.4, U1.3, U1.5; no longer J3.1
- net CAN_RX: now also U1.4; no longer J3.3
- net CAN_TX: now also U1.1; no longer J3.2
- net GND: now also J8.2, J8.3, U$5.GND, U1.2, U1.8; no longer J3.4
Routing:
- net GND: track 404.1 -> 0.00 mm, vias 3 -> 0
- net +5V: track 289.0 -> 0.00 mm, vias 5 -> 0
- net +15V: track 188.9 -> 0.00 mm, vias 4 -> 0
- net VCC: track 135.3 -> 0.00 mm, vias 3 -> 0
- net +3.3V: track 96.8 -> 0.00 mm
- net SCL_BUS: track 91.3 -> 0.00 mm, vias 2 -> 0
- net SDA_BUS: track 87.3 -> 0.00 mm, vias 3 -> 0
- net S_E: track 70.7 -> 0.00 mm
- net DIN: track 67.2 -> 0.00 mm
- net S_F: track 66.7 -> 0.00 mm
- net N$5: track 64.6 -> 0.00 mm
- net S_G: track 61.2 -> 0.00 mm, vias 2 -> 0
- net S_H: track 53.9 -> 0.00 mm, vias 3 -> 0
- net N$11: track 49.1 -> 0.00 mm
- net DOUT: track 48.0 -> 0.00 mm, vias 1 -> 0
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Other:
- board size 126 x 72 mm -> 135 x 72 mm
