File: processing_board/processing_board/schematic_v1.sch (EAGLE design)
At the start: 74 parts, among them J5 FEMALE 2x3, Q1 BSS138, Q2 BSS138, Q3 BSS138, Q4 BSS138, U1 SN74ALS166D

Commit message: added arduino
Parts:
- removed J6, J7: (no value), SparkFun-Connectors:CONN_08NO_SILK_FEMALE_PTH
- removed J8: (no value), SparkFun-Connectors:CONN_06SILK_FEMALE_PTH
- removed J9: (no value), SparkFun-Connectors:CONN_10"
- added AD, A_PWR: (no value), SparkFun-Connectors:CONN_06SILK_FEMALE_PTH
- added C7: 0.1uF, SparkFun-Capacitors:0.1UF-0603-25V-(+80/-20%)
- added IOH, IOL: (no value), SparkFun-Connectors:CONN_08NO_SILK_FEMALE_PTH
- added R33: 1k, SparkFun-Resistors:1KOHM-0603-1/10W-1%
- added R34: 10k, SparkFun-Resistors:1KOHM-0603-1/10W-1%
- added U2: ATMEGA328P_TQFP, SparkFun-IC-Microcontroller:ATMEGA328P_TQFP
- added U3: SN74HC595D, SparkFun-IC-Logic:74HC595D
- JP4: device pinhead:PINHD-1X1 -> pinhead:PINHD-2X3
Connections:
- net CAN_RX1 renamed SDA_BUS
- net CAN_TX1 renamed SCL_BUS
- new net A_AREF: IOH.8, U2.AREF
- new net A_MISO: IOH.5, JP4.1, U2.PB4(MISO)
- new net A_MOSI: IOH.4, JP4.4, U2.PB3(MOSI/OC2)
- new net A_RESET: A_PWR.1, JP4.5, R34.2, U2.PC6(/RESET)
- new net A_SCK: IOH.6, JP4.3, U2.PB5(SCK)
- new net A_SS: IOH.3, U2.PB2(SS/OC1B)
- new net N$26: JP1.11, U$4.33-MCLK2
- new net N$27: R33.1, U1.!CLR
- new net N$28: AD.1, U2.PC0(ADC0)
- new net N$29: AD.2, U2.PC1(ADC1)
- new net N$31: AD.3, U2.PC2(ADC2)
- new net N$32: AD.4, U2.PC3(ADC3)
- new net N$33: AD.5, U2.PC4(ADC4/SDA)
- new net N$34: AD.6, U2.PC5(ADC5/SCL)
- new net N$35: IOH.2, U2.PB1(OC1A)
- new net N$36: IOH.1, U2.PB0(ICP)
- new net N$37: IOL.8, U2.PD7(AIN1)
- new net N$38: IOL.7, U2.PD6(AIN0)
- new net N$39: IOL.6, U2.PD5(T1)
- new net N$40: IOL.5, U2.PD4(XCK/T0)
- new net N$41: IOL.4, U2.PD3(INT1)
- new net N$42: IOL.3, U2.PD2(INT0)
- new net N$43: IOL.2, U2.PD1(TXD)
- new net N$44: IOL.1, U2.PD0(RXD)
- new net N$50: A_PWR.6
- net +3.3V: now also A_PWR.2, JP1.3; no longer JP1.2
- net +5V: now also A_PWR.3, C7.1, JP4.2, R34.1, U2.AVCC, U2.VCC; no longer J6.1
- net GND: now also A_PWR.4, A_PWR.5, C7.2, IOH.7, JP1.12, JP1.14, JP1.2, JP4.6, U2.AGND, U2.GND; no longer J6.2, J6.3, JP1.11, JP1.13, JP4.1
- net N$1: now also JP1.5; no longer JP1.4
- net N$2: now also JP1.4; no longer JP1.3
- net N$3: now also JP1.13; no longer JP1.12
- net RESET_: now also JP1.7; no longer JP1.10, JP1.6, U$4.33-MCLK2
- net TEENSY_3.3V: now also R33.2; no longer U1.!CLR
Other:
- moved on the sheet: J5, JP1

Commit message: updated board
Parts:
- removed J1, J2: (no value), SparkFun-Connectors:BANANA_CONN
- removed U3: SN74HC595D, SparkFun-IC-Logic:74HC595D
- added BT1: (no value), SparkFun-Batteries:BATTERY-20MM_SMD
- added Y1: 16MHz, SparkFun-Clocks:RESONATOR-16MHZSMD_3.2X1.3
- J5: value FEMALE 2x3 -> (none); device SparkFun-Connectors:CONN_03X2FEMALE -> SparkFun-Connectors:CONN_02LOCK_LONGPADS
Connections:
- net N$28 renamed A_A0
- net N$44 renamed RXD
- removed net N$34: AD.6, U2.PC5(ADC5/SCL)
- new net N$45: U2.PB6(XTAL1/TOSC1), Y1.1
- new net N$46: U2.PB7(XTAL2/TOSC2), Y1.3
- net +15V: now also J5.1; no longer J1.1
- net GND: now also BT1.-, J5.2, Y1.2; no longer J2.1
- net N$33: now also BT1.+, U$4.VBAT; no longer AD.5, U2.PC4(ADC4/SDA)
- net SCL_BUS: now also AD.6, U2.PC5(ADC5/SCL)
- net SDA_BUS: now also AD.5, U2.PC4(ADC4/SDA)
Changed lines of the file:
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@@
 <part name="JP2" library="pinhead" library_urn="urn:adsk.eagle:library:325" deviceset="PINHD-1X8" device="" package3d_urn="urn:adsk.eagle:package:22409/2"/>
 <part name="GND1" library="supply" deviceset="GND" device=""/>
-<part name="J1" library="SparkFun-Connectors" deviceset="BANANA_CONN" device=""/>
-<part name="J2" library="SparkFun-Connectors" deviceset="BANANA_CONN" device=""/>
 <part name="GND2" library="supply" deviceset="GND" device=""/>
 <part name="PWR2" library="supply" deviceset="+15V" device=""/>
@@
 <part name="AD" library="SparkFun-Connectors" deviceset="CONN_06" device="SILK_FEMALE_PTH"/>
 <part name="IOH" library="SparkFun-Connectors" deviceset="CONN_08" device="NO_SILK_FEMALE_PTH"/>
-<part name="J5" library="SparkFun-Connectors" deviceset="CONN_03X2" device="FEMALE" value="FEMALE 2x3"/>
 <part name="S1" library="SparkFun-Switches" deviceset="DIP-08" device="-PTH"/>
 <part name="R20" library="SparkFun-Resistors" deviceset="10KOHM" device="-0603-1/10W-1%" value="10k"/>
@@
 <part name="U2" library="SparkFun-IC-Microcontroller" deviceset="ATMEGA328P_TQFP" device="" value="ATMEGA328P_TQFP"/>
 <part name="R33" library="SparkFun-Resistors" deviceset="1KOHM" device="-0603-1/10W-1%" value="1k"/>
-<part name="U3" library="SparkFun-IC-Logic" deviceset="74*595" device="D" technology="HC" value="SN74HC595D"/>
 <part name="IOL" library="SparkFun-Connectors" deviceset="CONN_08" device="NO_SILK_FEMALE_PTH"/>
 <part name="A_PWR" library="SparkFun-Connectors" deviceset="CONN_06" device="SILK_FEMALE_PTH"/>
@@
 <part name="C7" library="SparkFun-Capacitors" deviceset="0.1UF" device="-0603-25V-(+80/-20%)" value="0.1uF"/>
 <part name="PWR22" library="supply" deviceset="+5V" device=""/>
+<part name="Y1" library="SparkFun-Clocks" deviceset="RESONATOR-16MHZ" device="SMD_3.2X1.3" value="16MHz"/>
+<part name="BT1" library="SparkFun-Batteries" deviceset="BATTERY" device="-20MM_SMD"/>
+<part name="J5" library="SparkFun-Connectors" deviceset="CONN_02" device="LOCK_LONGPADS"/>
 </parts>
 <sheets>
@@
 </instance>
 <instance part="GND1" gate="VR1" x="33.02" y="-15.24" smashed="yes"/>
-<instance part="J1" gate="G$1" x="106.68" y="167.64" smashed="yes" grouprefs="POWER">
-<attribute name="NAME" x="105.664" y="169.418" size="1.778" layer="95" font="vector"/>
-<attribute name="VALUE" x="105.664" y="164.592" size="1.778" layer="96" font="vector"/>
-</instance>
-<instance part="J2" gate="G$1" x="106.68" y="162.56" smashed="yes" grouprefs="POWER">
-<attribute name="NAME" x="105.664" y="164.338" size="1.778" layer="95" font="vector"/>
-<attribute name="VALUE" x="105.664" y="159.512" size="1.778" layer="96" font="vector"/>
-</instance>
 <instance part="GND2" gate="VR1" x="101.6" y="157.48" smashed="yes" grouprefs="POWER"/>
 <instance part="PWR2" gate="G$1" x="99.06" y="172.72" smashed="yes" grouprefs="POWER"/>
@@
 <attribute name="NAME" x="307.34" y="-79.248" size="1.778" layer="95" font="vector" rot="R180"/>
 </instance>
-<instance part="J5" gate="G$1" x="248.92" y="-101.6" smashed="yes" rot="R90">
-<attribute name="NAME" x="243.332" y="-105.156" size="1.778" layer="95" font="vector" rot="R90"/>
-<attribute name="VALUE" x="254.762" y="-104.902" size="1.778" layer="96" font="vector" rot="R90" align="top-left"/>
-</instance>
 <instance part="S1" gate="A" x="33.02" y="-91.44" smashed="yes">
 <attribute name="NAME" x="33.02" y="-81.026" size="1.778" layer="95" font="vector" align="bottom-center"/>
@@
 <attribute name="NAME" x="139.7" y="-133.096" size="1.778" layer="95" font="vector" align="bottom-center"/>
 <attribute name="VALUE" x="139.7" y="-136.144" size="1.778" layer="96" font="vector" align="top-center"/>
-</instance>
-<instance part="U3" gate="U1" x="162.56" y="-15.24" smashed="yes">
-<attribute name="NAME" x="157.48" y="-1.778" size="1.778" layer="95" font="vector"/>
-<attribute name="VALUE" x="157.48" y="-33.02" size="1.778" layer="95" font="vector"/>
 </instance>
 <instance part="IOL" gate="G$1" x="289.56" y="-40.64" smashed="yes" rot="R180">
@@
 </instance>
 <instance part="PWR22" gate="G$1" x="198.12" y="-20.32" smashed="yes"/>
+<instance part="Y1" gate="G$1" x="226.06" y="-38.1" smashed="yes" rot="R270">
+<attribute name="NAME" x="223.52" y="-34.798" size="1.778" layer="95" font="vector" rot="R270" align="center-right"/>
+<attribute name="VALUE" x="228.092" y="-38.1" size="1.778" layer="96" font="vector" rot="R270" align="bottom-center"/>
+</instance>
+<instance part="BT1" gate="G$1" x="60.96" y="-7.62" smashed="yes" rot="R270">
+<attribute name="NAME" x="65.278" y="-7.62" size="1.778" layer="95" font="vector" rot="R270" align="bottom-center"/>
+<attribute name="VALUE" x="56.642" y="-7.62" size="1.778" layer="96" font="vector" rot="R270" align="top-center"/>
+</instance>
+<instance part="J5" gate="G$1" x="114.3" y="165.1" smashed="yes" rot="R180">
+<attribute name="VALUE" x="116.84" y="169.926" size="1.778" layer="96" font="vector" rot="R180"/>
+<attribute name="NAME" x="116.84" y="159.512" size="1.778" layer="95" font="vector" rot="R180"/>
+</instance>
 </instances>
 <busses>
@@
 </segment>
 <segment>
-<pinref part="J2" gate="G$1" pin="1"/>
 <pinref part="GND2" gate="VR1" pin="GND"/>
-<wire x1="104.14" y1="162.56" x2="101.6" y2="162.56" width="0.1524" layer="91" grouprefs="POWER"/>
+<wire x1="106.68" y1="162.56" x2="101.6" y2="162.56" width="0.1524" layer="91" grouprefs="POWER"/>
 <wire x1="101.6" y1="162.56" x2="101.6" y2="160.02" width="0.1524" layer="91" grouprefs="POWER"/>
+<pinref part="J5" gate="G$1" pin="2"/>
 </segment>
 <segment>
@@
 <label x="198.12" y="-30.48" size="1.778" layer="95"/>
 </segment>
+<segment>
+<pinref part="Y1" gate="G$1" pin="2"/>
+<wire x1="218.44" y1="-38.1" x2="213.36" y2="-38.1" width="0.1524" layer="91"/>
+<label x="213.36" y="-38.1" size="1.778" layer="95"/>
+</segment>
+<segment>
+<pinref part="BT1" gate="G$1" pin="-"/>
+<wire x1="60.96" y1="-12.7" x2="60.96" y2="-17.78" width="0.1524" layer="91"/>
+<label x="60.96" y="-17.78" size="1.778" layer="95"/>
+</segment>
 </net>
 <net name="+15V" class="0">
 <segment>
-<pinref part="J1" gate="G$1" pin="1"/>
 <pinref part="PWR2" gate="G$1" pin="+15V"/>
 <wire x1="104.14" y1="167.64" x2="99.06" y2="167.64" width="0.1524" layer="91" grouprefs="POWER"/>
 <wire x1="99.06" y1="167.64" x2="99.06" y2="172.72" width="0.1524" layer="91" grouprefs="POWER"/>
 <wire x1="104.14" y1="167.64" x2="104.14" y2="175.26" width="0.1524" layer="91"/>
-<junction x="104.14" y="167.64"/>
 <wire x1="104.14" y1="175.26" x2="137.16" y2="175.26" width="0.1524" layer="91"/>
 <wire x1="137.16" y1="175.26" x2="137.16" y2="170.18" width="0.1524" layer="91"/>
 <pinref part="R18" gate="G$1" pin="2"/>
+<wire x1="104.14" y1="167.64" x2="104.14" y2="165.1" width="0.1524" layer="91"/>
+<junction x="104.14" y="167.64"/>
+<pinref part="J5" gate="G$1" pin="1"/>
+<wire x1="104.14" y1="165.1" x2="106.68" y2="165.1" width="0.1524" layer="91"/>
 </segment>
 <segment>
@@
 <label x="284.48" y="43.18" size="1.778" layer="95"/>
 </segment>
+<segment>
+<pinref part="U2" gate="U1" pin="PC4(ADC4/SDA)"/>
+<pinref part="AD" gate="G$1" pin="5"/>
+<wire x1="276.86" y1="-20.32" x2="304.8" y2="-20.32" width="0.1524" layer="91"/>
+<label x="287.02" y="-20.32" size="1.778" layer="95"/>
+</segment>
 </net>
 <net name="SCL_BUS" class="0">
@@
 <label x="284.48" y="45.72" size="1.778" layer="95"/>
 </segment>
+<segment>
+<pinref part="U2" gate="U1" pin="PC5(ADC5/SCL)"/>
+<pinref part="AD" gate="G$1" pin="6"/>
+<wire x1="276.86" y1="-22.86" x2="304.8" y2="-22.86" width="0.1524" layer="91"/>
+<label x="287.02" y="-22.86" size="1.778" layer="95"/>
+</segment>
 </net>
 <net name="N$4" class="0">
@@
 </segment>
 </net>
-<net name="N$28" class="0">
+<net name="A_A0" class="0">
 <segment>
 <pinref part="U2" gate="U1" pin="PC0(ADC0)"/>
 <pinref part="AD" gate="G$1" pin="1"/>
 <wire x1="276.86" y1="-10.16" x2="304.8" y2="-10.16" width="0.1524" layer="91"/>
+<label x="281.94" y="-10.16" size="1.778" layer="95"/>
 </segment>
 </net>
@@
 <pinref part="AD" gate="G$1" pin="4"/>
 <wire x1="276.86" y1="-17.78" x2="304.8" y2="-17.78" width="0.1524" layer="91"/>
-</segment>
-</net>
-<net name="N$33" class="0">
-<segment>
-<pinref part="U2" gate="U1" pin="PC4(ADC4/SDA)"/>
-<pinref part="AD" gate="G$1" pin="5"/>
-<wire x1="276.86" y1="-20.32" x2="304.8" y2="-20.32" width="0.1524" layer="91"/>
-</segment>
-</net>
-<net name="N$34" class="0">
-<segment>
-<pinref part="U2" gate="U1" pin="PC5(ADC5/SCL)"/>
-<pinref part="AD" gate="G$1" pin="6"/>
-<wire x1="276.86" y1="-22.86" x2="304.8" y2="-22.86" width="0.1524" layer="91"/>
 </segment>
 </net>
@@
 </segment>
 </net>
-<net name="N$44" class="0">
+<net name="RXD" class="0">
 <segment>
 <pinref part="IOL" gate="G$1" pin="1"/>
 <pinref part="U2" gate="U1" pin="PD0(RXD)"/>
 <wire x1="284.48" y1="-33.02" x2="276.86" y2="-33.02" width="0.1524" layer="91"/>
+<label x="279.4" y="-33.02" size="1.778" layer="95"/>
 </segment>
 </net>
@@
 </segment>
 </net>
+<net name="N$45" class="0">
+<segment>
+<pinref part="Y1" gate="G$1" pin="1"/>
+<pinref part="U2" gate="U1" pin="PB6(XTAL1/TOSC1)"/>
+<wire x1="226.06" y1="-35.56" x2="233.68" y2="-35.56" width="0.1524" layer="91"/>
+</segment>
+</net>
+<net name="N$46" class="0">
+<segment>
+<pinref part="U2" gate="U1" pin="PB7(XTAL2/TOSC2)"/>
+<pinref part="Y1" gate="G$1" pin="3"/>
+<wire x1="233.68" y1="-40.64" x2="226.06" y2="-40.64" width="0.1524" layer="91"/>
+</segment>
+</net>
+<net name="N$33" class="0">
+<segment>
+<pinref part="U$4" gate="G$1" pin="VBAT"/>
+<pinref part="BT1" gate="G$1" pin="+"/>
+<wire x1="55.88" y1="7.62" x2="60.96" y2="7.62" width="0.1524" layer="91"/>
+<wire x1="60.96" y1="7.62" x2="60.96" y2="-2.54" width="0.1524" layer="91"/>
+</segment>
+</net>

Commit message: finished wiring
Parts:
- removed JP2: (no value), pinhead:PINHD-1X8
Changed lines of the file:
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@@
 </groups>
 <parts>
-<part name="JP2" library="pinhead" library_urn="urn:adsk.eagle:library:325" deviceset="PINHD-1X8" device="" package3d_urn="urn:adsk.eagle:package:22409/2"/>
 <part name="GND1" library="supply" deviceset="GND" device=""/>
 <part name="GND2" library="supply" deviceset="GND" device=""/>
@@
 </plain>
 <instances>
-<instance part="JP2" gate="A" x="-154.94" y="-53.34" smashed="yes" rot="MR90">
-<attribute name="NAME" x="-141.605" y="-59.69" size="1.778" layer="95" rot="MR90"/>
-<attribute name="VALUE" x="-167.64" y="-59.69" size="1.778" layer="96" rot="MR90"/>
-</instance>
 <instance part="GND1" gate="VR1" x="33.02" y="-15.24" smashed="yes"/>
 <instance part="GND2" gate="VR1" x="101.6" y="157.48" smashed="yes" grouprefs="POWER"/>

Commit message: generated gerber files
Parts:
- removed B1: ARDUINO_UNO_R3, SparkFun-Boards:ARDUINO_UNO_R3
Connections:
- removed net N$19: B1.GND
Changed lines of the file:
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@@
 <part name="GND14" library="supply" deviceset="GND" device=""/>
 <part name="U$4" library="teensy" deviceset="TEENSY41-E" device=""/>
-<part name="B1" library="SparkFun-Boards" deviceset="ARDUINO_UNO_R3" device=""/>
 <part name="R18" library="SparkFun-Resistors" deviceset="10KOHM" device="-0603-1/10W-1%" value="10k"/>
 <part name="R19" library="SparkFun-Resistors" deviceset="8.2KOHM" device="-0603-1/10W-5%" value="8.2k"/>
@@
 <instance part="GND14" gate="VR1" x="-187.96" y="-22.86" smashed="yes" rot="MR90"/>
 <instance part="U$4" gate="G$1" x="25.4" y="35.56" smashed="yes" rot="MR0"/>
-<instance part="B1" gate="G$1" x="142.24" y="58.42" smashed="yes">
-<attribute name="NAME" x="132.588" y="89.662" size="1.778" layer="95" font="vector"/>
-<attribute name="VALUE" x="132.08" y="27.686" size="1.778" layer="96" font="vector" align="top-left"/>
-</instance>
 <instance part="R18" gate="G$1" x="137.16" y="165.1" smashed="yes" rot="R90">
 <attribute name="NAME" x="135.636" y="165.1" size="1.778" layer="95" font="vector" rot="R90" align="bottom-center"/>
@@
 <segment>
 <wire x1="129.54" y1="30.48" x2="130.81" y2="30.48" width="0.1524" layer="91"/>
-<pinref part="B1" gate="G$1" pin="GND"/>
-</segment>
-</net>
+</segment>
+</net>
