File: processing_board/processing_board/schematic_v1.sch (EAGLE design)
At the start: 70 parts, among them IC1 74HC165D, Q1 BSS138, Q2 BSS138, Q3 BSS138, Q4 BSS138, U1 TJA1050

Commit message: v3 update
Parts:
- removed IC1: 74HC165D, 74xx-eu:74HC165D
- removed J3, J6: (no value), SparkFun-Connectors:CONN_08"
- removed J7, J8: (no value), SparkFun-Connectors:CONN_06NO_SILK_FEMALE_PTH
- added CN1: (no value), adafruit:DCBARRELPTH
- added J2: (no value), SparkFun-Connectors:I2C_STANDARD
- added JP1, JP2: (no value), pinhead:PINHD-1X4
- added R33: 10k, SparkFun-Resistors:10KOHM-0603-1/10W-1%
- added S2: (no value), SparkFun-Switches:MOMENTARY-SWITCH-SPST-2-SMD-5.2MM
Connections:
- net N$1 renamed CAN_L
- net N$2 renamed CAN_H
- new net IN_A: S2.3, S2.4, U$4.26-A12/MOSI1
- new net N$2: R33.1
- net +15V: now also CN1.PWR
- net +3.3V: now also JP2.1; no longer J8.5
- net +5V: now also J2.2, JP1.1, S1.10, S1.11, S1.12, S1.13, S1.14, S1.15, S1.16, S1.9, S2.1, S2.2; no longer J8.1, J8.4, U1.VREF
- net CAN_RX: now also JP1.3
- net CAN_TX: now also JP1.2
- net CLK_INH: no longer IC1A.INH
- net DIN: now also JP2.3
- net DIP_SW_SERIAL: no longer IC1A.QH
- net DOUT: now also JP2.2
- net GND: now also CN1.GND, J2.1, JP1.4, JP2.4, R20.1, R26.1, R27.1, R30.1, R31.1, R32.1, R33.2; no longer IC1A.SER, J8.2, J8.3
- net LS_CK: no longer IC1A.CLK
- net N$23: no longer R20.1, R26.1, R27.1, R30.1, R31.1, R32.1
- net SCL_BUS: now also J2.4
- net SDA_BUS: now also J2.3
- net SH_LD: no longer IC1A.SH/!LD
- net S_A: now also U$4.18-A4/SDA0; no longer IC1A.A
- net S_B: now also U$4.19-A5/SCL0; no longer IC1A.B
- net S_C: now also U$4.20-A6/TX5/LRCLK1; no longer IC1A.C
- net S_D: now also U$4.21-A7/RX5/BCLK1; no longer IC1A.D
- net S_E: now also U$4.22-A8/CTX1; no longer IC1A.E
- net S_F: now also U$4.23-A9/CRX1/MCLK1; no longer IC1A.F
- net S_G: now also U$4.24-A10/TX6/SCL2; no longer IC1A.G
- net S_H: now also U$4.25-A11/RX6/SDA2; no longer IC1A.H
- net VCC: no longer S1.10, S1.11, S1.12, S1.13, S1.14, S1.15, S1.16, S1.9
Other:
- moved on the sheet: D8, R17, R20, R26, R27, R28, R29, R30, R31, R32, S1
